Commit message: Edited urdf/yamls, fixed lifecycle manager

File: src/my_robot_bringup/urdf/robo_cayote.urdf (robot description, URDF)
Before this commit: robot robo_cayote, 34 links, 33 joints
Links:
- added link base_footprint
- link base_link: geometry collision box size=0.45 0.31 0.06; visual box size=0.45 0.31 0.06
- link solid_1: geometry collision cylinder length=0.08 radius=0.095; visual cylinder length=0.08 radius=0.095
- link solid_13: geometry collision cylinder length=0.08 radius=0.095; visual cylinder length=0.08 radius=0.095
- link solid_5: geometry collision cylinder length=0.08 radius=0.095; visual cylinder length=0.08 radius=0.095
- link solid_9: geometry collision cylinder length=0.08 radius=0.095; visual cylinder length=0.08 radius=0.095
Joints:
- added joint base_footprint_joint: type fixed, parent base_footprint, child base_link, origin xyz=0 0 0.26 rpy=0 0 0
- joint base_link_to_camera: origin xyz=0 0.28 0 rpy=0 0 0 -> xyz=0 0 0.29 rpy=0 0 0
- joint base_link_ultrasonic_front_joint: origin xyz=0.38 0.05 0 rpy=0 0 0 -> xyz=0.215 0 0.03 rpy=0 0 0
- joint base_link_ultrasonic_front_left_joint: origin xyz=0.33 0.05 0.18 rpy=0 0 0 -> xyz=0.205 0.12 0.03 rpy=0 0 .785
- joint base_link_ultrasonic_front_right_joint: origin xyz=0.33 0.05 -0.18 rpy=0 0 0 -> xyz=0.205 -0.12 0.03 rpy=0 0 -.785
- joint base_link_ultrasonic_rear_joint: origin xyz=-0.38 0.05 0 rpy=0 3.14159 0 -> xyz=-0.215 0 0.03 rpy=0 0 3.14159
- joint base_link_ultrasonic_rear_left_joint: origin xyz=-0.33 0.05 0.18 rpy=0 3.14159 0 -> xyz=-0.205 0.12 0.03 rpy=0 0 2.35659
- joint base_link_ultrasonic_rear_right_joint: origin xyz=-0.33 0.05 -0.18 rpy=0 3.14159 0 -> xyz=-0.205 -0.12 0.03 rpy=0 0 3.92659
- joint base_link_ultrasonic_side_left_back_joint: origin xyz=-0.20 0.05 0.22 rpy=0 -1.5708 0 -> xyz=-0.12 0.14 0.03 rpy=0 0 1.5708
- joint base_link_ultrasonic_side_left_front_joint: origin xyz=0.20 0.05 0.22 rpy=0 -1.5708 0 -> xyz=0.09 0.14 0.03 rpy=0 0 1.5708
- joint base_link_ultrasonic_side_right_back_joint: origin xyz=-0.20 0.05 -0.22 rpy=0 1.5708 0 -> xyz=-0.09 -0.14 0.03 rpy=0 0 -1.5708
- joint base_link_ultrasonic_side_right_front_joint: origin xyz=0.20 0.05 -0.22 rpy=0 1.5708 0 -> xyz=0.12 -0.14 0.03 rpy=0 0 -1.5708
- joint sliderjoint: axis 0 1 0 -> 0 0 1; origin xyz=0.31 0.02 -0.28 rpy=0 0 0 -> xyz=0.31 -0.17 -0.165 rpy=0 0 0
- joint sliderjoint_11: axis 0 1 0 -> 0 0 1; origin xyz=-0.31 0.02 0.28 rpy=0 0 0 -> xyz=-0.31 0.17 -0.165 rpy=0 0 0
- joint sliderjoint_2: axis 0 1 0 -> 0 0 1; origin xyz=0.31 0.02 0.28 rpy=0 0 0 -> xyz=0.31 0.17 -0.165 rpy=0 0 0
- joint sliderjoint_7: axis 0 1 0 -> 0 0 1; origin xyz=-0.31 0.02 -0.28 rpy=0 0 0 -> xyz=-0.31 -0.17 -0.165 rpy=0 0 0
- joint steer_motor_fl: axis 0 1 0 -> 0 0 1
- joint steer_motor_fr: axis 0 1 0 -> 0 0 1
- joint wheel_motor_fl: axis 0 0 1 -> 0 1 0
- joint wheel_motor_fr: axis 0 0 1 -> 0 1 0
- joint wheel_motor_rl: axis 0 0 1 -> 0 1 0
- joint wheel_motor_rr: axis 0 0 1 -> 0 1 0
