Commit message: Update robo_cayote_des.urdf

File: Webots_Files/robo_cayote_des.urdf (robot description, URDF)
Before this commit: robot robo_cayote, 9 links, 8 joints
Links:
- added link appearance, mass 0.01; visual box size=0.001 0.001 0.001
- added link appearance_10, mass 0.01; visual box size=0.001 0.001 0.001
- added link appearance_14, mass 0.01; visual box size=0.001 0.001 0.001
- added link appearance_15, mass 0.01; visual box size=0.001 0.001 0.001
- added link appearance_6, mass 0.01; visual box size=0.001 0.001 0.001
- added link base_footprint, mass 0.01; visual box size=0.001 0.001 0.001
- added link camera_left_frame, mass 0.01; visual box size=0.001 0.001 0.001
- added link camera_left_optical_frame, mass 0.01; visual box size=0.001 0.001 0.001
- added link camera_link, mass 0.01; visual box size=0.001 0.001 0.001
- added link camera_right_frame, mass 0.01; visual box size=0.001 0.001 0.001
- added link camera_right_optical_frame, mass 0.01; visual box size=0.001 0.001 0.001
- added link compass, mass 0.01; visual box size=0.001 0.001 0.001
- added link solid_12, mass 0.01; visual box size=0.001 0.001 0.001
- added link solid_13, mass 0.5; collision cylinder length=0.08 radius=0.095; visual cylinder length=0.08 radius=0.095
- added link solid_8, mass 0.01; visual box size=0.001 0.001 0.001
- added link solid_9, mass 0.5; collision cylinder length=0.08 radius=0.095; visual cylinder length=0.08 radius=0.095
- added link ultrasonic_front_left_link, mass 0.01; visual box size=0.001 0.001 0.001
- added link ultrasonic_front_link, mass 0.01; visual box size=0.001 0.001 0.001
- added link ultrasonic_front_right_link, mass 0.01; visual box size=0.001 0.001 0.001
- added link ultrasonic_rear_left_link, mass 0.01; visual box size=0.001 0.001 0.001
- added link ultrasonic_rear_link, mass 0.01; visual box size=0.001 0.001 0.001
- added link ultrasonic_rear_right_link, mass 0.01; visual box size=0.001 0.001 0.001
- added link ultrasonic_side_left_back_link, mass 0.01; visual box size=0.001 0.001 0.001
- added link ultrasonic_side_left_front_link, mass 0.01; visual box size=0.001 0.001 0.001
- added link ultrasonic_side_right_back_link, mass 0.01; visual box size=0.001 0.001 0.001
- added link ultrasonic_side_right_front_link, mass 0.01; visual box size=0.001 0.001 0.001
- link base_link: geometry collision box size=0.45 0.31 0.06; visual box size=0.45 0.31 0.06
- link solid_1: geometry collision cylinder length=0.08 radius=0.095; visual cylinder length=0.08 radius=0.095
- link solid_5: geometry collision cylinder length=0.08 radius=0.095; visual cylinder length=0.08 radius=0.095
Joints:
- removed joint base_gps
- removed joint base_imu
- removed joint slider_fl
- removed joint slider_fr
- added joint base_footprint_joint: type fixed, parent base_footprint, child base_link, origin xyz=0 0 0.26 rpy=0 0 0
- added joint base_link_appearance_15_joint: type fixed, parent base_link, child appearance_15, origin xyz=0 0 0 rpy=0 0 0
- added joint base_link_compass_joint: type fixed, parent base_link, child compass, origin xyz=0 0 0 rpy=0 0 0
- added joint base_link_gps_joint: type fixed, parent base_link, child gps, origin xyz=0 0 0 rpy=0 0 0
- added joint base_link_imu_joint: type fixed, parent base_link, child imu, origin xyz=0 0 0 rpy=0 0 0
- added joint base_link_to_camera: type fixed, parent base_link, child camera_link, origin xyz=0 0 0.29 rpy=0 0 0
- added joint base_link_ultrasonic_front_joint: type fixed, parent base_link, child ultrasonic_front_link, origin xyz=0.215 0 0.03 rpy=0 0 0
- added joint base_link_ultrasonic_front_left_joint: type fixed, parent base_link, child ultrasonic_front_left_link, origin xyz=0.205 0.12 0.03 rpy=0 0 .785
- added joint base_link_ultrasonic_front_right_joint: type fixed, parent base_link, child ultrasonic_front_right_link, origin xyz=0.205 -0.12 0.03 rpy=0 0 -.785
- added joint base_link_ultrasonic_rear_joint: type fixed, parent base_link, child ultrasonic_rear_link, origin xyz=-0.215 0 0.03 rpy=0 0 3.14159
- added joint base_link_ultrasonic_rear_left_joint: type fixed, parent base_link, child ultrasonic_rear_left_link, origin xyz=-0.205 0.12 0.03 rpy=0 0 2.35659
- added joint base_link_ultrasonic_rear_right_joint: type fixed, parent base_link, child ultrasonic_rear_right_link, origin xyz=-0.205 -0.12 0.03 rpy=0 0 3.92659
- added joint base_link_ultrasonic_side_left_back_joint: type fixed, parent base_link, child ultrasonic_side_left_back_link, origin xyz=-0.12 0.14 0.03 rpy=0 0 1.5708
- added joint base_link_ultrasonic_side_left_front_joint: type fixed, parent base_link, child ultrasonic_side_left_front_link, origin xyz=0.09 0.14 0.03 rpy=0 0 1.5708
- added joint base_link_ultrasonic_side_right_back_joint: type fixed, parent base_link, child ultrasonic_side_right_back_link, origin xyz=-0.09 -0.14 0.03 rpy=0 0 -1.5708
- added joint base_link_ultrasonic_side_right_front_joint: type fixed, parent base_link, child ultrasonic_side_right_front_link, origin xyz=0.12 -0.14 0.03 rpy=0 0 -1.5708
- added joint camera_left_joint: type fixed, parent camera_link, child camera_left_frame, origin xyz=0 0.025 0 rpy=0 0 0
- added joint camera_left_optical_joint: type fixed, parent camera_left_frame, child camera_left_optical_frame, origin xyz=0 0 0 rpy=-1.5708 0 -1.5708
- added joint camera_right_joint: type fixed, parent camera_link, child camera_right_frame, origin xyz=0 -0.025 0 rpy=0 0 0
- added joint camera_right_optical_joint: type fixed, parent camera_right_frame, child camera_right_optical_frame, origin xyz=0 0 0 rpy=-1.5708 0 -1.5708
- added joint sliderjoint: type prismatic, parent base_link, child solid, origin xyz=0.31 -0.17 -0.165 rpy=0 0 0, axis 0 0 1, limit lower=-0.1 upper=0.1 effort=10 velocity=10
- added joint sliderjoint_11: type prismatic, parent base_link, child solid_12, origin xyz=-0.31 0.17 -0.165 rpy=0 0 0, axis 0 0 1, limit lower=-0.1 upper=0.1 effort=10 velocity=10
- added joint sliderjoint_2: type prismatic, parent base_link, child solid_3, origin xyz=0.31 0.17 -0.165 rpy=0 0 0, axis 0 0 1, limit lower=-0.1 upper=0.1 effort=10 velocity=10
- added joint sliderjoint_7: type prismatic, parent base_link, child solid_8, origin xyz=-0.31 -0.17 -0.165 rpy=0 0 0, axis 0 0 1, limit lower=-0.1 upper=0.1 effort=10 velocity=10
- added joint solid_13_appearance_14_joint: type fixed, parent solid_13, child appearance_14, origin xyz=0 0 0 rpy=0 0 0
- added joint solid_1_appearance_joint: type fixed, parent solid_1, child appearance, origin xyz=0 0 0 rpy=0 0 0
- added joint solid_5_appearance_6_joint: type fixed, parent solid_5, child appearance_6, origin xyz=0 0 0 rpy=0 0 0
- added joint solid_9_appearance_10_joint: type fixed, parent solid_9, child appearance_10, origin xyz=0 0 0 rpy=0 0 0
- added joint wheel_motor_rl: type continuous, parent solid_12, child solid_13, origin xyz=0 0 0 rpy=0 0 0, axis 0 1 0, limit effort=20 velocity=10
- added joint wheel_motor_rr: type continuous, parent solid_8, child solid_9, origin xyz=0 0 0 rpy=0 0 0, axis 0 1 0, limit effort=20 velocity=10
- joint steer_motor_fl: axis 0 1 0 -> 0 0 1; limit (none) -> effort=5 velocity=10; origin (none) -> xyz=0 0 0 rpy=0 0 0
- joint steer_motor_fr: axis 0 1 0 -> 0 0 1; limit (none) -> effort=5 velocity=10; origin xyz=0 0 0 -> xyz=0 0 0 rpy=0 0 0
- joint wheel_motor_fl: axis 0 0 1 -> 0 1 0; limit (none) -> effort=20 velocity=10; origin (none) -> xyz=0 0 0 rpy=0 0 0
- joint wheel_motor_fr: axis 0 0 1 -> 0 1 0; limit (none) -> effort=20 velocity=10; origin xyz=0 0 0 -> xyz=0 0 0 rpy=0 0 0
